File: schematic/operational-fanifier-schematic.sch (KiCad schematic (older format))
At the start: 17 parts, among them M1 Fan, Q1 BC337, Q2 BC337, SW1 SW_SPDT, U1 LM324N, U2 74HC32, U3 LM335Z

Commit message: Mostly-final layouted schematic
Parts:
- removed R?: 1MRTRIM, symbol Device:RTRIM
- removed unit 1 of U1
- added C4: 10nF, Capacitor_SMD:C_0805_2012Metric, symbol Device:C
- added J1: Conn_01x03, Connector_PinHeader_2.54mm:PinHeader_1x03_P2.54mm_Horizontal, symbol Connector_Generic:Conn_01x03
- added RV2: 1MR_POT, Potentiometer_THT:Potentiometer_Bourns_3266Y_Vertical, symbol Device:R_POT
- added unit 4 of U1
- added unit 3 of U1
- C1, C2: footprint (none) -> Capacitor_SMD:C_0805_2012Metric
- C3: footprint (none) -> Capacitor_THT:CP_Radial_D5.0mm_P2.50mm
- M1: footprint (none) -> Connector_PinHeader_2.54mm:PinHeader_1x02_P2.54mm_Vertical
- Q1, Q2: footprint Package_TO_SOT_THT:TO-92_Inline -> Package_TO_SOT_THT:TO-92_Inline_Wide
- R1, R2, R4, R5: footprint (none) -> Resistor_THT:R_Axial_DIN0204_L3.6mm_D1.6mm_P5.08mm_Horizontal
- R3: footprint (none) -> Resistor_THT:R_Axial_DIN0204_L3.6mm_D1.6mm_P7.62mm_Horizontal
- RV1: value R_POT -> 5kR_POT; footprint (none) -> Potentiometer_THT:Potentiometer_Bourns_3266Y_Vertical
- SW1, U3: footprint (none) -> Connector_PinHeader_2.54mm:PinHeader_1x03_P2.54mm_Vertical
- U1, U2: footprint (none) -> Package_DIP:DIP-14_W7.62mm
Connections:
- wire segments 11 -> 14
Other:
- note added: "(for board layout use only)"
- moved on the sheet: U1E
