File: schematic/operational-fanifier-schematic.sch (KiCad schematic (older format))
At the start: 19 parts, among them J1 Conn_01x03, M1 Fan, Q1 BC337, Q2 BC337, SW1 SW_SPDT, U1 LM324N, U2 74HC32, U3 LM335Z

Commit message: I really should think these things through
Parts:
- M1: footprint Connector_PinHeader_2.54mm:PinHeader_1x02_P2.54mm_Horizontal -> Connector_PinHeader_2.54mm:PinHeader_2x01_P2.54mm_Vertical_SMD
Changed lines of the file:
@@
 F 0 "M1" H 4408 4996 50  0000 L CNN
 F 1 "Fan" H 4408 4905 50  0000 L CNN
-F 2 "Connector_PinHeader_2.54mm:PinHeader_1x02_P2.54mm_Horizontal" H 4250 4910 50  0001 C CNN
+F 2 "Connector_PinHeader_2.54mm:PinHeader_2x01_P2.54mm_Vertical_SMD" H 4250 4910 50  0001 C CNN
 F 3 "~" H 4250 4910 50  0001 C CNN
 	1    4250 4900
