File: schematic/operational-fanifier-schematic.kicad_pcb (KiCad board)
At the start: 2 copper layers, 19 parts, among them J1 Conn_01x03, M1 Fan, Q1 BC337, Q2 BC337, SW1 SW_SPDT, U1 LM324N, U2 74HC32, U3 LM335Z

Commit message: I really should think these things through
Parts:
- M1: footprint Connector_PinHeader_2.54mm:PinHeader_1x02_P2.54mm_Horizontal -> Connector_PinHeader_2.54mm:PinHeader_2x01_P2.54mm_Vertical_SMD; moved to B.Cu
- moved M1 1.27 mm to (158.8, 26.7), turned to 270 degrees
Changed lines of the file:
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@@
-    )
-  )
-  (module Connector_PinHeader_2.54mm:PinHeader_1x02_P2.54mm_Horizontal (layer F.Cu)
-    (at 158.75 25.4)
-    (descr "Through hole angled pin header, 1x02, 2.54mm pitch, 6mm pin length, single row")
-    (tags "Through hole angled pin header THT 1x02 2.54mm single row")
-    (fp_text reference M1 (at 4.385 -2.27) (layer F.SilkS)
-      (effects (font (size 1 1) (thickness 0.15)))
-    )
-    (fp_text value Fan (at 4.385 4.81) (layer F.Fab)
-      (effects (font (size 1 1) (thickness 0.15)))
-    )
-    (fp_line (start 2.135 -1.27) (end 4.04 -1.27) (layer F.Fab) (width 0.1))
-    (fp_line (start 4.04 -1.27) (end 4.04 3.81) (layer F.Fab) (width 0.1))
-    (fp_line (start 4.04 3.81) (end 1.5 3.81) (layer F.Fab) (width 0.1))
-    (fp_line (start 1.5 3.81) (end 1.5 -0.635) (layer F.Fab) (width 0.1))
-    (fp_line (start 1.5 -0.635) (end 2.135 -1.27) (layer F.Fab) (width 0.1))
-    (fp_line (start -0.32 -0.32) (end 1.5 -0.32) (layer F.Fab) (width 0.1))
-    (fp_line (start -0.32 -0.32) (end -0.32 0.32) (layer F.Fab) (width 0.1))
-    (fp_line (start -0.32 0.32) (end 1.5 0.32) (layer F.Fab) (width 0.1))
-    (fp_line (start 4.04 -0.32) (end 10.04 -0.32) (layer F.Fab) (width 0.1))
-    (fp_line (start 10.04 -0.32) (end 10.04 0.32) (layer F.Fab) (width 0.1))
-    (fp_line (start 4.04 0.32) (end 10.04 0.32) (layer F.Fab) (width 0.1))
-    (fp_line (start -0.32 2.22) (end 1.5 2.22) (layer F.Fab) (width 0.1))
-    (fp_line (start -0.32 2.22) (end -0.32 2.86) (layer F.Fab) (width 0.1))
-    (fp_line (start -0.32 2.86) (end 1.5 2.86) (layer F.Fab) (width 0.1))
-    (fp_line (start 4.04 2.22) (end 10.04 2.22) (layer F.Fab) (width 0.1))
-    (fp_line (start 10.04 2.22) (end 10.04 2.86) (layer F.Fab) (width 0.1))
-    (fp_line (start 4.04 2.86) (end 10.04 2.86) (layer F.Fab) (width 0.1))
-    (fp_line (start 1.44 -1.33) (end 1.44 3.87) (layer F.SilkS) (width 0.12))
-    (fp_line (start 1.44 3.87) (end 4.1 3.87) (layer F.SilkS) (width 0.12))
-    (fp_line (start 4.1 3.87) (end 4.1 -1.33) (layer F.SilkS) (width 0.12))
-    (fp_line (start 4.1 -1.33) (end 1.44 -1.33) (layer F.SilkS) (width 0.12))
-    (fp_line (start 4.1 -0.38) (end 10.1 -0.38) (layer F.SilkS) (width 0.12))
-    (fp_line (start 10.1 -0.38) (end 10.1 0.38) (layer F.SilkS) (width 0.12))
-    (fp_line (start 10.1 0.38) (end 4.1 0.38) (layer F.SilkS) (width 0.12))
-    (fp_line (start 4.1 -0.32) (end 10.1 -0.32) (layer F.SilkS) (width 0.12))
-    (fp_line (start 4.1 -0.2) (end 10.1 -0.2) (layer F.SilkS) (width 0.12))
-    (fp_line (start 4.1 -0.08) (end 10.1 -0.08) (layer F.SilkS) (width 0.12))
-    (fp_line (start 4.1 0.04) (end 10.1 0.04) (layer F.SilkS) (width 0.12))
-    (fp_line (start 4.1 0.16) (end 10.1 0.16) (layer F.SilkS) (width 0.12))
-    (fp_line (start 4.1 0.28) (end 10.1 0.28) (layer F.SilkS) (width 0.12))
-    (fp_line (start 1.11 -0.38) (end 1.44 -0.38) (layer F.SilkS) (width 0.12))
-    (fp_line (start 1.11 0.38) (end 1.44 0.38) (layer F.SilkS) (width 0.12))
-    (fp_line (start 1.44 1.27) (end 4.1 1.27) (layer F.SilkS) (width 0.12))
-    (fp_line (start 4.1 2.16) (end 10.1 2.16) (layer F.SilkS) (width 0.12))
-    (fp_line (start 10.1 2.16) (end 10.1 2.92) (layer F.SilkS) (width 0.12))
-    (fp_line (start 10.1 2.92) (end 4.1 2.92) (layer F.SilkS) (width 0.12))
-    (fp_line (start 1.042929 2.16) (end 1.44 2.16) (layer F.SilkS) (width 0.12))
-    (fp_line (start 1.042929 2.92) (end 1.44 2.92) (layer F.SilkS) (width 0.12))
-    (fp_line (start -1.27 0) (end -1.27 -1.27) (layer F.SilkS) (width 0.12))
-    (fp_line (start -1.27 -1.27) (end 0 -1.27) (layer F.SilkS) (width 0.12))
-    (fp_line (start -1.8 -1.8) (end -1.8 4.35) (layer F.CrtYd) (width 0.05))
-    (fp_line (start -1.8 4.35) (end 10.55 4.35) (layer F.CrtYd) (width 0.05))
-    (fp_line (start 10.55 4.35) (end 10.55 -1.8) (layer F.CrtYd) (width 0.05))
-    (fp_line (start 10.55 -1.8) (end -1.8 -1.8) (layer F.CrtYd) (width 0.05))
-    (fp_text user %R (at 2.77 1.27 90) (layer F.Fab)
-      (effects (font (size 1 1) (thickness 0.15)))
-    )
-    (pad 1 thru_hole rect (at 0 0) (size 1.7 1.7) (drill 1) (layers *.Cu *.Mask)
-      (net 5 +12V))
-    (pad 2 thru_hole oval (at 0 2.54) (size 1.7 1.7) (drill 1) (layers *.Cu *.Mask)
-      (net 18 "Net-(M1-Pad2)"))
-    (model ${KISYS3DMOD}/Connector_PinHeader_2.54mm.3dshapes/PinHeader_1x02_P2.54mm_Horizontal.wrl
-      (at (xyz 0 0 0))
-      (scale (xyz 1 1 1))
-      (rotate (xyz 0 0 0))
     )
   )
@@
       (at (xyz 0 0 0))
       (scale (xyz 1 1 1))
+      (rotate (xyz 0 0 0))
+    )
+  )
+  (module Connector_PinHeader_2.54mm:PinHeader_2x01_P2.54mm_Vertical_SMD (layer B.Cu)
+    (at 158.75 26.67 270)
+    (descr "surface-mounted straight pin header, 2x01, 2.54mm pitch, double rows")
+    (tags "Surface mounted pin header SMD 2x01 2.54mm double row")
+    (attr smd)
+    (fp_text reference M1 (at 0 2.33 270) (layer B.SilkS)
+      (effects (font (size 1 1) (thickness 0.15)) (justify mirror))
+    )
+    (fp_text value Fan (at 0 -2.33 270) (layer B.Fab)
+      (effects (font (size 1 1) (thickness 0.15)) (justify mirror))
+    )
+    (fp_line (start 2.54 -1.27) (end -2.54 -1.27) (layer B.Fab) (width 0.1))
+    (fp_line (start -1.59 1.27) (end 2.54 1.27) (layer B.Fab) (width 0.1))
+    (fp_line (start -2.54 -1.27) (end -2.54 0.32) (layer B.Fab) (width 0.1))
+    (fp_line (start -2.54 0.32) (end -1.59 1.27) (layer B.Fab) (width 0.1))
+    (fp_line (start 2.54 1.27) (end 2.54 -1.27) (layer B.Fab) (width 0.1))
+    (fp_line (start -2.54 0.32) (end -3.6 0.32) (layer B.Fab) (width 0.1))
+    (fp_line (start -3.6 0.32) (end -3.6 -0.32) (layer B.Fab) (width 0.1))
+    (fp_line (start -3.6 -0.32) (end -2.54 -0.32) (layer B.Fab) (width 0.1))
+    (fp_line (start 2.54 0.32) (end 3.6 0.32) (layer B.Fab) (width 0.1))
+    (fp_line (start 3.6 0.32) (end 3.6 -0.32) (layer B.Fab) (width 0.1))
+    (fp_line (start 3.6 -0.32) (end 2.54 -0.32) (layer B.Fab) (width 0.1))
+    (fp_line (start -2.6 1.33) (end 2.6 1.33) (layer B.SilkS) (width 0.12))
+    (fp_line (start -2.6 -1.33) (end 2.6 -1.33) (layer B.SilkS) (width 0.12))
+    (fp_line (start -4.04 0.76) (end -2.6 0.76) (layer B.SilkS) (width 0.12))
+    (fp_line (start -2.6 1.33) (end -2.6 0.76) (layer B.SilkS) (width 0.12))
+    (fp_line (start 2.6 1.33) (end 2.6 0.76) (layer B.SilkS) (width 0.12))
+    (fp_line (start -2.6 -0.76) (end -2.6 -1.33) (layer B.SilkS) (width 0.12))
+    (fp_line (start 2.6 -0.76) (end 2.6 -1.33) (layer B.SilkS) (width 0.12))
+    (fp_line (start -5.9 1.8) (end -5.9 -1.8) (layer B.CrtYd) (width 0.05))
+    (fp_line (start -5.9 -1.8) (end 5.9 -1.8) (layer B.CrtYd) (width 0.05))
+    (fp_line (start 5.9 -1.8) (end 5.9 1.8) (layer B.CrtYd) (width 0.05))
+    (fp_line (start 5.9 1.8) (end -5.9 1.8) (layer B.CrtYd) (width 0.05))
+    (fp_text user %R (at 0 0 180) (layer B.Fab)
+      (effects (font (size 1 1) (thickness 0.15)) (justify mirror))
+    )
+    (pad 1 smd rect (at -2.525 0 270) (size 3.15 1) (layers B.Cu B.Paste B.Mask)
+      (net 5 +12V))
+    (pad 2 smd rect (at 2.525 0 270) (size 3.15 1) (layers B.Cu B.Paste B.Mask)
+      (net 18 "Net-(M1-Pad2)"))
+    (model ${KISYS3DMOD}/Connector_PinHeader_2.54mm.3dshapes/PinHeader_2x01_P2.54mm_Vertical_SMD.wrl
+      (at (xyz 0 0 0))
+      (scale (xyz 1 1 1))
